File: ldr_contr.sch (KiCad schematic (older format))
At the start: 15 parts, among them U1 ADG728, U2 ADG728, U3 ADG728, U5 LM317_3PinPackage

Commit message: schematic finalized
Parts:
- U4: renamed from U?; symbol PCA9306 -> PCA9306-RESCUE-ldr_contr
- gave numbers to parts that had none: 3
Connections:
- net labels removed: 5.5V
- wire segments 96 -> 199
- no-connect marks 0 -> 6
Other:
- moved on the sheet: U4

Commit message: board ready
Parts:
- added Rp4, Rp5: 4.7k, Resistors_ThroughHole:Resistor_Horizontal_RM10mm, symbol R
- C1, C2: footprint (none) -> Capacitors_ThroughHole:C_Radial_D6.3_L11.2_P2.5
- P1: footprint (none) -> Connect:PINHEAD1-3
- P2: footprint (none) -> created:PINHEAD1-4
- P3: footprint (none) -> Connect:IDC_Header_Straight_34pins
- R1, R2, Rp1, Rp2, Rp3: footprint (none) -> Resistors_ThroughHole:Resistor_Horizontal_RM10mm
- U1, U2, U3: footprint (none) -> Housings_SSOP:TSSOP-16_4.4x5mm_Pitch0.65mm
- U4: footprint (none) -> Housings_SOIC:SO-8_5.3x6.2mm_Pitch1.27mm
- U5: footprint (none) -> Power_Integrations:TO-220
Connections:
- net SCL: now also P1.3 (P3), Rp4.2; no longer P1.1 (P1)
- net at P2.3 (P3), U4.2 (Vref1): now also Rp4.1, Rp5.2
- net SDA: no longer names the net of U4.5 (SDA2)
- net SDA: now also P1.1 (P1), Rp5.1; no longer P1.3 (P3)
Changed lines of the file:
@@
 F 0 "U1" H 4900 2400 50  0000 C CNN
 F 1 "ADG728" H 4900 900 50  0000 C CNN
-F 2 "" H 4900 1650 60  0001 C CNN
+F 2 "Housings_SSOP:TSSOP-16_4.4x5mm_Pitch0.65mm" H 4900 1650 60  0001 C CNN
 F 3 "" H 4900 1650 60  0001 C CNN
 	1    4900 1650
@@
 F 0 "U2" H 4850 6400 50  0000 C CNN
 F 1 "ADG728" H 4850 4900 50  0000 C CNN
-F 2 "" H 4850 5650 60  0001 C CNN
+F 2 "Housings_SSOP:TSSOP-16_4.4x5mm_Pitch0.65mm" H 4850 5650 60  0001 C CNN
 F 3 "" H 4850 5650 60  0001 C CNN
 	1    4850 5650
@@
 F 0 "U3" H 4850 4550 50  0000 C CNN
 F 1 "ADG728" H 4850 3050 50  0000 C CNN
-F 2 "" H 4850 3800 60  0001 C CNN
+F 2 "Housings_SSOP:TSSOP-16_4.4x5mm_Pitch0.65mm" H 4850 3800 60  0001 C CNN
 F 3 "" H 4850 3800 60  0001 C CNN
 	1    4850 3800
@@
 F 0 "U5" H 1550 6425 50  0000 C CNN
 F 1 "LM317_3PinPackage" H 1700 6425 50  0000 L CNN
-F 2 "" H 1700 6550 50  0001 C CIN
+F 2 "Power_Integrations:TO-220" H 1700 6550 50  0001 C CIN
 F 3 "" H 1700 6300 50  0001 C CNN
 	1    1700 6300
@@
 F 0 "R1" V 1780 7200 50  0000 C CNN
 F 1 "287R" V 1700 7200 50  0000 C CNN
-F 2 "" V 1630 7200 50  0001 C CNN
+F 2 "Resistors_ThroughHole:Resistor_Horizontal_RM10mm" V 1630 7200 50  0001 C CNN
 F 3 "" H 1700 7200 50  0001 C CNN
 	1    1700 7200
@@
 F 0 "R2" V 1330 6750 50  0000 C CNN
 F 1 "1kR" V 1250 6750 50  0000 C CNN
-F 2 "" V 1180 6750 50  0001 C CNN
+F 2 "Resistors_ThroughHole:Resistor_Horizontal_RM10mm" V 1180 6750 50  0001 C CNN
 F 3 "" H 1250 6750 50  0001 C CNN
 	1    1250 6750
@@
 F 0 "C1" H 2225 6700 50  0000 L CNN
 F 1 "100uF / 25V" H 2225 6500 50  0000 L CNN
-F 2 "" H 2238 6450 50  0001 C CNN
+F 2 "Capacitors_ThroughHole:C_Radial_D6.3_L11.2_P2.5" H 2238 6450 50  0001 C CNN
 F 3 "" H 2200 6600 50  0001 C CNN
 	1    2200 6600
@@
 F 0 "C2" H 925 6800 50  0000 L CNN
 F 1 "100uF / 25V" H 925 6600 50  0000 L CNN
-F 2 "" H 938 6550 50  0001 C CNN
+F 2 "Capacitors_ThroughHole:C_Radial_D6.3_L11.2_P2.5" H 938 6550 50  0001 C CNN
 F 3 "" H 900 6700 50  0001 C CNN
 	1    900  6700
@@
 F 0 "P3" H 2000 4800 50  0000 C CNN
 F 1 "CONN_02X17" V 2000 3900 50  0000 C CNN
-F 2 "" H 2000 2800 50  0000 C CNN
+F 2 "Connect:IDC_Header_Straight_34pins" H 2000 2800 50  0001 C CNN
 F 3 "" H 2000 2800 50  0000 C CNN
 	1    2000 3900
@@
 F 0 "P1" H 10550 3300 50  0000 C CNN
 F 1 "CONN_01X03" V 10650 3100 50  0000 C CNN
-F 2 "" H 10550 3100 50  0000 C CNN
+F 2 "Connect:PINHEAD1-3" H 10550 3100 50  0001 C CNN
 F 3 "" H 10550 3100 50  0000 C CNN
 	1    10550 3100
-	1    0    0    -1
+	1    0    0    1
 $EndComp
 $Comp
@@
 F 0 "Rp1" V 7080 4250 50  0000 C CNN
 F 1 "4.7k" V 7000 4250 50  0000 C CNN
-F 2 "" V 6930 4250 50  0000 C CNN
+F 2 "Resistors_ThroughHole:Resistor_Horizontal_RM10mm" V 6930 4250 50  0001 C CNN
 F 3 "" H 7000 4250 50  0000 C CNN
 	1    7000 4250
@@
 F 0 "Rp2" V 7530 4250 50  0000 C CNN
 F 1 "4.7k" V 7450 4250 50  0000 C CNN
-F 2 "" V 7380 4250 50  0000 C CNN
+F 2 "Resistors_ThroughHole:Resistor_Horizontal_RM10mm" V 7380 4250 50  0001 C CNN
 F 3 "" H 7450 4250 50  0000 C CNN
 	1    7450 4250
@@
 F 0 "U4" H 8250 2250 60  0000 C CNN
 F 1 "PCA9306" H 8250 2950 60  0000 C CNN
-F 2 "" H 8150 2850 60  0000 C CNN
+F 2 "Housings_SOIC:SO-8_5.3x6.2mm_Pitch1.27mm" H 8150 2850 60  0001 C CNN
 F 3 "" H 8150 2850 60  0000 C CNN
 	1    8250 2800
@@
 F 0 "P2" H 10400 6050 50  0000 C CNN
 F 1 "CONN_01X04" V 10500 5800 50  0000 C CNN
-F 2 "" H 10400 5800 50  0000 C CNN
+F 2 "created:PINHEAD1-4" H 10400 5800 50  0001 C CNN
 F 3 "" H 10400 5800 50  0000 C CNN
 	1    10400 5800
@@
 	7900 2600 7900 2850
 Wire Wire Line
-	9700 5000 7950 5000
+	7950 5000 10800 5000
 Wire Wire Line
 	7950 5000 7950 3450
@@
 F 0 "Rp3" V 8830 2200 50  0000 C CNN
 F 1 "200k" V 8750 2200 50  0000 C CNN
-F 2 "" V 8680 2200 50  0000 C CNN
+F 2 "Resistors_ThroughHole:Resistor_Horizontal_RM10mm" V 8680 2200 50  0001 C CNN
 F 3 "" H 8750 2200 50  0000 C CNN
 	1    8750 2200
@@
 Text Label 10000 3000 0    60   ~ 0
 SCL
-Text Label 10000 3200 0    60   ~ 0
-SDA
 Wire Wire Line
 	900  3800 900  6550
@@
 NoConn ~ 2250 4700
 NoConn ~ 1750 4700
+$Comp
+L R Rp4
+U 1 1 5ACDCB15
+P 9850 2850
+F 0 "Rp4" V 9930 2850 50  0000 C CNN
+F 1 "4.7k" V 9850 2850 50  0000 C CNN
+F 2 "Resistors_ThroughHole:Resistor_Horizontal_RM10mm" V 9780 2850 50  0001 C CNN
+F 3 "" H 9850 2850 50  0000 C CNN
+	1    9850 2850
+	1    0    0    -1
+$EndComp
+$Comp
+L R Rp5
+U 1 1 5ACDCBB0
+P 9850 3350
+F 0 "Rp5" V 9930 3350 50  0000 C CNN
+F 1 "4.7k" V 9850 3350 50  0000 C CNN
+F 2 "Resistors_ThroughHole:Resistor_Horizontal_RM10mm" V 9780 3350 50  0001 C CNN
+F 3 "" H 9850 3350 50  0000 C CNN
+	1    9850 3350
+	1    0    0    -1
+$EndComp
+Wire Wire Line
+	9850 5000 9850 3500
+Wire Wire Line
+	10800 5000 10800 2700
+Wire Wire Line
+	10800 2700 9850 2700
+Connection ~ 9850 5000
+Connection ~ 9850 3000
+Connection ~ 9850 3200
 $EndSCHEMATC

Commit message: cleanup
Parts:
- removed P3: CONN_02X17, Connect:IDC_Header_Straight_34pins, symbol CONN_02X17
- removed U4: PCA9306, Housings_SOIC:SO-8_5.3x6.2mm_Pitch1.27mm, symbol PCA9306-RESCUE-ldr_contr
- added J2: Conn_02x17_Odd_Even, Connect:IDC_Header_Straight_34pins, symbol Conn_02x17_Odd_Even
- added U4: PCA9306, Housings_SOIC:SOIC-8_3.9x4.9mm_Pitch1.27mm, symbol PCA9306
- P1: symbol CONN_01X03 -> Conn_01x03
- P2: symbol CONN_01X04 -> Conn_01x04
- renumbered U3 to U2, U2 to U3
Connections:
- net GND: now also J2.17 (Pin_17), J2.18 (Pin_18), U4.1 (GND)
- net SCL: now also U4.6 (SCL2)
- net at Rp2.2, U1.1 (SCL), U2.1 (SCL)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: now also U4.3 (SCL1)
- net at U1.10 (S7): now also J2.4 (Pin_4)
- net at U1.11 (S6): now also J2.3 (Pin_3)
- net at U1.12 (S5): now also J2.5 (Pin_5)
- net at P2.1 (Pin_1), Rp1.1, Rp2.1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: now also Rp3.2; no longer Rp3.1
- net at Rp1.2, U1.3 (SDA), U2.3 (SDA)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: now also U4.4 (SDA1)
- net at U1.4 (S1): now also J2.13 (Pin_13)
- net at U1.5 (S2): now also J2.11 (Pin_11)
- net at U1.6 (S3): now also J2.9 (Pin_9)
- net at U1.7 (S4): now also J2.7 (Pin_7)
- net at U1.9 (S8): now also J2.6 (Pin_6)
- net at U3.10 (S7): now also J2.23 (Pin_23)
- net at U3.11 (S6): now also J2.25 (Pin_25)
- net at U3.12 (S5): now also J2.27 (Pin_27)
- net at U3.4 (S1): now also J2.30 (Pin_30)
- net at U3.5 (S2): now also J2.32 (Pin_32)
- net at U3.6 (S3): now also J2.31 (Pin_31)
- net at U3.7 (S4): now also J2.29 (Pin_29)
- net at U3.9 (S8): now also J2.21 (Pin_21)
- net at U2.10 (S7): now also J2.26 (Pin_26)
- net at U2.11 (S6): now also J2.24 (Pin_24)
- net at U2.12 (S5): now also J2.22 (Pin_22)
- net at U2.4 (S1): now also J2.8 (Pin_8)
- net at U2.5 (S2): now also J2.10 (Pin_10)
- net at U2.6 (S3): now also J2.12 (Pin_12)
- net at U2.7 (S4): now also J2.14 (Pin_14)
- net at U2.9 (S8): now also J2.28 (Pin_28)
- net at C2.1, R2.1, U5.2 (VO): now also J2.19 (Pin_19), J2.20 (Pin_20)
- net at P1.1 (Pin_1), Rp5.1: now also U4.5 (SDA2)
- net at P2.3 (Pin_3), Rp4.1, Rp5.2: now also U4.2 (VREF1)
- new net: Rp3.1, U4.7 (VREF2), U4.8 (EN)
Other:
- moved on the sheet: Rp3
Changed lines of the file:
@@
 LIBS:valves
 LIBS:ti
-LIBS:ldr_contr-cache
 EELAYER 25 0
 EELAYER END
@@
 $EndComp
 $Comp
-L ADG728 U2
+L ADG728 U3
 U 1 1 5ACA145F
 P 4850 5650
-F 0 "U2" H 4850 6400 50  0000 C CNN
+F 0 "U3" H 4850 6400 50  0000 C CNN
 F 1 "ADG728" H 4850 4900 50  0000 C CNN
 F 2 "Housings_SSOP:TSSOP-16_4.4x5mm_Pitch0.65mm" H 4850 5650 60  0001 C CNN
@@
 $EndComp
 $Comp
-L ADG728 U3
+L ADG728 U2
 U 1 1 5ACA14CB
 P 4850 3800
-F 0 "U3" H 4850 4550 50  0000 C CNN
+F 0 "U2" H 4850 4550 50  0000 C CNN
 F 1 "ADG728" H 4850 3050 50  0000 C CNN
 F 2 "Housings_SSOP:TSSOP-16_4.4x5mm_Pitch0.65mm" H 4850 3800 60  0001 C CNN
@@
 Connection ~ 900  6300
 $Comp
-L CONN_02X17 P3
-U 1 1 5ACC571B
-P 2000 3900
-F 0 "P3" H 2000 4800 50  0000 C CNN
-F 1 "CONN_02X17" V 2000 3900 50  0000 C CNN
-F 2 "Connect:IDC_Header_Straight_34pins" H 2000 2800 50  0001 C CNN
-F 3 "" H 2000 2800 50  0000 C CNN
-	1    2000 3900
-	-1   0    0    1
-$EndComp
-$Comp
 L +9V #PWR03
 U 1 1 5ACC57CF
@@
 Connection ~ 5550 3350
 $Comp
-L CONN_01X03 P1
+L Conn_01x03 P1
 U 1 1 5ACC634F
 P 10550 3100
@@
 	4300 5050 4300 4850
 Wire Wire Line
-	8600 3200 10350 3200
-Wire Wire Line
 	4300 5150 4200 5150
 Wire Wire Line
 	4200 5150 4200 4750
 Wire Wire Line
-	8700 3000 10350 3000
+	9750 3000 10350 3000
 Wire Wire Line
 	4300 3200 4300 2950
@@
 	3600 700  3600 5400
 $Comp
-L PCA9306-RESCUE-ldr_contr U4
-U 1 1 5ACC8C6F
-P 8250 2800
-F 0 "U4" H 8250 2250 60  0000 C CNN
-F 1 "PCA9306" H 8250 2950 60  0000 C CNN
-F 2 "Housings_SOIC:SO-8_5.3x6.2mm_Pitch1.27mm" H 8150 2850 60  0001 C CNN
-F 3 "" H 8150 2850 60  0000 C CNN
-	1    8250 2800
-	1    0    0    -1
-$EndComp
-$Comp
-L CONN_01X04 P2
+L Conn_01x04 P2
 U 1 1 5ACC8DCA
-P 10400 5800
-F 0 "P2" H 10400 6050 50  0000 C CNN
-F 1 "CONN_01X04" V 10500 5800 50  0000 C CNN
-F 2 "created:PINHEAD1-4" H 10400 5800 50  0001 C CNN
-F 3 "" H 10400 5800 50  0000 C CNN
-	1    10400 5800
+P 10400 5750
+F 0 "P2" H 10400 6000 50  0000 C CNN
+F 1 "CONN_01X04" V 10500 5750 50  0000 C CNN
+F 2 "created:PINHEAD1-4" H 10400 5750 50  0001 C CNN
+F 3 "" H 10400 5750 50  0000 C CNN
+	1    10400 5750
 	1    0    0    -1
 $EndComp
@@
 	7600 4750 7600 3150
 Wire Wire Line
-	7600 3150 7900 3150
-Connection ~ 7600 4750
+	7600 3150 6750 3150
 Wire Wire Line
 	4200 4750 7600 4750
@@
 	4300 4850 7750 4850
 Wire Wire Line
-	7750 4850 7750 3050
-Wire Wire Line
-	7750 3050 7900 3050
-Wire Wire Line
-	8700 3000 8700 3050
-Wire Wire Line
-	8700 3050 8600 3050
-Wire Wire Line
-	8600 3200 8600 3150
-Wire Wire Line
-	9200 2600 7900 2600
-Wire Wire Line
-	7900 2600 7900 2850
-Wire Wire Line
 	7950 5000 10800 5000
 Wire Wire Line
-	7950 5000 7950 3450
-Wire Wire Line
-	7950 3450 7450 3450
-Wire Wire Line
-	7450 3450 7450 2950
-Wire Wire Line
-	7450 2950 7900 2950
+	7950 3450 7950 5000
+Wire Wire Line
+	6500 3450 7950 3450
 Connection ~ 9700 5000
 $Comp
 L R Rp3
 U 1 1 5ACC9DFB
-P 8750 2200
-F 0 "Rp3" V 8830 2200 50  0000 C CNN
-F 1 "200k" V 8750 2200 50  0000 C CNN
-F 2 "Resistors_ThroughHole:Resistor_Horizontal_RM10mm" V 8680 2200 50  0001 C CNN
-F 3 "" H 8750 2200 50  0000 C CNN
-	1    8750 2200
-	1    0    0    -1
-$EndComp
-Wire Wire Line
-	8600 2350 8600 2950
-Wire Wire Line
-	8600 2350 8750 2350
-Connection ~ 8600 2850
+P 8200 1750
+F 0 "Rp3" V 8280 1750 50  0000 C CNN
+F 1 "200k" V 8200 1750 50  0000 C CNN
+F 2 "Resistors_ThroughHole:Resistor_Horizontal_RM10mm" V 8130 1750 50  0001 C CNN
+F 3 "" H 8200 1750 50  0000 C CNN
+	1    8200 1750
+	0    -1   -1   0
+$EndComp
 Wire Wire Line
 	8750 2050 11050 2050
@@
 Connection ~ 9850 3000
 Connection ~ 9850 3200
+$Comp
+L Conn_02x17_Odd_Even J2
+U 1 1 5ACFB191
+P 2050 3900
+F 0 "J2" H 2100 4800 50  0000 C CNN
+F 1 "Conn_02x17_Odd_Even" H 2100 3000 50  0000 C CNN
+F 2 "Connect:IDC_Header_Straight_34pins" H 2050 3900 50  0001 C CNN
+F 3 "" H 2050 3900 50  0001 C CNN
+	1    2050 3900
+	-1   0    0    1
+$EndComp
+$Comp
+L PCA9306 U4
+U 1 1 5ACFBC9F
+P 7650 1850
+F 0 "U4" H 7350 2300 50  0000 L CNN
+F 1 "PCA9306" H 7850 2300 50  0000 L CNN
+F 2 "Housings_SOIC:SOIC-8_3.9x4.9mm_Pitch1.27mm" H 7250 2200 50  0001 C CNN
+F 3 "" H 7350 2300 50  0001 C CNN
+	1    7650 1850
+	1    0    0    -1
+$EndComp
+Wire Wire Line
+	7750 1350 8050 1350
+Wire Wire Line
+	8050 1350 8050 1750
+Wire Wire Line
+	8750 2050 8750 1750
+Wire Wire Line
+	8750 1750 8350 1750
+Wire Wire Line
+	9200 2600 7650 2600
+Wire Wire Line
+	7650 2600 7650 2350
+Wire Wire Line
+	9750 3000 9750 2150
+Wire Wire Line
+	9750 2150 8600 2150
+Wire Wire Line
+	8600 2150 8600 1850
+Wire Wire Line
+	8600 1850 8050 1850
+Wire Wire Line
+	9650 3200 9650 2300
+Wire Wire Line
+	9650 2300 8500 2300
+Wire Wire Line
+	8500 2300 8500 1950
+Wire Wire Line
+	8500 1950 8050 1950
+Connection ~ 9650 3200
+Wire Wire Line
+	9650 3200 10350 3200
+Wire Wire Line
+	7750 4850 7750 2650
+Wire Wire Line
+	7750 2650 6650 2650
+Wire Wire Line
+	6650 2650 6650 1850
+Wire Wire Line
+	6650 1850 7250 1850
+Wire Wire Line
+	6750 3150 6750 1950
+Wire Wire Line
+	6750 1950 7250 1950
+Wire Wire Line
+	6500 3450 6500 1200
+Wire Wire Line
+	6500 1200 7550 1200
+Wire Wire Line
+	7550 1200 7550 1350
 $EndSCHEMATC

Commit message: kicad update to version 5, ADG728 is now using the defualt Library
Parts:
- C1, C2: symbol CP -> Device:CP
- J2: symbol Conn_02x17_Odd_Even -> Connector_Generic:Conn_02x17_Odd_Even
- P1: symbol Conn_01x03 -> Connector_Generic:Conn_01x03
- P2: symbol Conn_01x04 -> Connector_Generic:Conn_01x04
- R1, R2, Rp1, Rp2, Rp3, Rp4, Rp5: symbol R -> Device:R
- U1, U2, U3: footprint Housings_SSOP:TSSOP-16_4.4x5mm_Pitch0.65mm -> Package_SO:TSSOP-16_4.4x5mm_P0.65mm; symbol ADG728 -> Analog_Switch:ADG728
- U4: symbol PCA9306 -> Interface:PCA9306
- U5: symbol LM317_3PinPackage -> Regulator_Linear:LM317_3PinPackage
Connections:
- wire segments 214 -> 267
Other:
- moved on the sheet: U3
